File: pcb/kitritiled.kicad_pcb (KiCad board)
At the start: 4 copper layers, 22.8 x 22.8 mm, 15 parts, among them J1 ICSP, J2 ICSP, Q1 AO3401A, Q2 AO3400A, SW1 RESET, U1 PIC12LF1571-I/SN, U2 74LVC1G123

Commit message: updates
Parts:
- moved R1 9.18 mm to (85.0, 85.7)
- moved C1 1.80 mm to (92.0, 93.5)
- moved C2 1.80 mm to (93.5, 93.5)
- moved U1 1.07 mm to (96.9, 90.1)
- turned BT1 to 180 degrees
- turned R2 to 180 degrees
Routing:
- net +3V0: track 0.00 -> 34.6 mm, vias 0 -> 2
- net Net-(BT1-+): track 0.00 -> 24.2 mm, vias 0 -> 2
- net CLR: track 0.00 -> 16.8 mm, vias 0 -> 2
- net Net-(SW1-A): track 0.00 -> 16.6 mm
- net Net-(U1-RA4): track 0.00 -> 14.9 mm, vias 0 -> 2
- net Net-(D1-A): track 0.00 -> 13.2 mm
- net GND: track 0.00 -> 12.1 mm, vias 0 -> 5
- net Net-(Q2-G): track 0.00 -> 7.34 mm
- net Net-(U2A-RCext): track 0.00 -> 6.53 mm
- net ICSP_DATA: track 0.00 -> 5.94 mm
- net ICSP_CLK: track 0.00 -> 3.93 mm
- net Net-(Q1-G): track 0.00 -> 3.48 mm
- net Net-(U2A-Cext): track 0.00 -> 2.04 mm
- added copper zone on B.Cu, net GND
Other:
- copper layers 4 -> 2

Commit message: license and silkscreen
Other:
- board text added: "<<hash>>"
- board text added: "kitritiled v1"
Changed lines of the file:
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@@
     (property "ki_keywords" "battery cell")
     (attr smd)
-    (fp_text reference "BT1" (at 0 -6) (layer "B.SilkS")
+    (fp_text reference "BT1" (at 0 -6) (layer "B.SilkS") hide
         (effects (font (size 1 1) (thickness 0.15)) (justify mirror))
     )
@@
   (gr_circle (center 90 90) (end 101.4 90)
     (stroke (width 0.1) (type default)) (fill none) (layer "Edge.Cuts"))
+  (gr_text "<<hash>>" (at 90 100) (layer "B.SilkS")
+    (effects (font (size 0.8 0.8) (thickness 0.12)) (justify mirror))
+  )
+  (gr_text "kitritiled\nv1" (at 90 80.5) (layer "F.SilkS")
+    (effects (font (size 0.8 0.8) (thickness 0.12)))
+  )
   (segment (start 94.2625 94.275) (end 93.5 94.275) (width 0.2) (layer "F.Cu") (net 1))
   (segment (start 89.902137 88.502137) (end 83.252137 88.502137) (width 0.2) (layer "F.Cu") (net 1))

Commit message: nudge
Parts:
- moved L1 0.49 mm to (83.0, 90.0)
Routing:
- net +3V0: track 34.6 -> 33.7 mm
- net Net-(D1-A): track 13.2 -> 12.5 mm
Changed lines of the file:
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@@
   )
   (footprint "Inductor_SMD:L_Sunlord_SWPA6028S" (layer "F.Cu")
-    (at 82.5 90 -90)
+    (at 82.9861 89.999999 -90)
     (descr "Inductor, Sunlord, SWPA6028S, 6.0x6.0x2.8mm, https://www.sunlordinc.com/UploadFiles/PDF_Cat/20120704094224784.pdf")
     (tags "Inductor swpa")
@@
   )
   (segment (start 94.2625 94.275) (end 93.5 94.275) (width 0.2) (layer "F.Cu") (net 1))
-  (segment (start 89.902137 88.502137) (end 83.252137 88.502137) (width 0.2) (layer "F.Cu") (net 1))
-  (segment (start 83.252137 88.502137) (end 82.5 87.75) (width 0.2) (layer "F.Cu") (net 1))
+  (segment (start 84.262538 89.026437) (end 82.9861 87.749999) (width 0.2) (layer "F.Cu") (net 1))
+  (segment (start 84.262538 90.507969) (end 84.262538 89.026437) (width 0.2) (layer "F.Cu") (net 1))
   (segment (start 94.15861 94.275) (end 95.03075 93.40286) (width 0.2) (layer "F.Cu") (net 1))
   (segment (start 93.5 94.275) (end 94.15861 94.275) (width 0.2) (layer "F.Cu") (net 1))
-  (segment (start 84.484556 85.665532) (end 84.484556 85.765444) (width 0.3) (layer "F.Cu") (net 1))
   (segment (start 82.703949 83.884925) (end 84.484556 85.665532) (width 0.3) (layer "F.Cu") (net 1))
   (segment (start 95.03075 93.40286) (end 95.03075 92.55966) (width 0.2) (layer "F.Cu") (net 1))
+  (segment (start 90 88.6) (end 89.902137 88.502137) (width 0.2) (layer "F.Cu") (net 1))
+  (segment (start 84.484556 85.665532) (end 84.484556 86.251543) (width 0.3) (layer "F.Cu") (net 1))
   (segment (start 82.703949 83.796051) (end 82.703949 83.884925) (width 0.3) (layer "F.Cu") (net 1))
   (segment (start 92 94.275) (end 93.5 94.275) (width 0.2) (layer "F.Cu") (net 1))
+  (segment (start 89.902137 88.502137) (end 83.738238 88.502137) (width 0.2) (layer "F.Cu") (net 1))
+  (segment (start 84.484556 86.251543) (end 82.9861 87.749999) (width 0.3) (layer "F.Cu") (net 1))
   (segment (start 84.873293 93.88) (end 84.861682 93.868389) (width 0.2) (layer "F.Cu") (net 1))
-  (segment (start 84.484556 85.765444) (end 82.5 87.75) (width 0.3) (layer "F.Cu") (net 1))
   (segment (start 91.605 93.88) (end 84.873293 93.88) (width 0.2) (layer "F.Cu") (net 1))
-  (segment (start 90 88.6) (end 89.902137 88.502137) (width 0.2) (layer "F.Cu") (net 1))
+  (segment (start 83.738238 88.502137) (end 82.9861 87.749999) (width 0.2) (layer "F.Cu") (net 1))
   (segment (start 95.55 95.5625) (end 94.2625 94.275) (width 0.2) (layer "F.Cu") (net 1))
   (segment (start 92 94.275) (end 91.605 93.88) (width 0.2) (layer "F.Cu") (net 1))
-  (segment (start 84.262538 90.507969) (end 84.262538 89.512538) (width 0.2) (layer "F.Cu") (net 1))
-  (segment (start 84.262538 89.512538) (end 82.5 87.75) (width 0.2) (layer "F.Cu") (net 1))
   (via (at 84.861682 93.868389) (size 0.6) (drill 0.4) (layers "F.Cu" "B.Cu") (net 1))
   (via (at 84.262538 90.507969) (size 0.6) (drill 0.4) (layers "F.Cu" "B.Cu") (net 1))
@@
   (segment (start 90.879179 95.222977) (end 93.145509 95.222977) (width 0.2) (layer "F.Cu") (net 4))
   (segment (start 93.55 96.675) (end 92.15 96.675) (width 0.2) (layer "F.Cu") (net 4))
-  (segment (start 84 93.75) (end 84 97) (width 0.3) (layer "F.Cu") (net 5))
-  (segment (start 83.239115 91.510885) (end 82.5 92.25) (width 0.2) (layer "F.Cu") (net 5))
-  (segment (start 82.5 92.25) (end 84 93.75) (width 0.3) (layer "F.Cu") (net 5))
+  (segment (start 82.9861 92.249999) (end 84 93.263899) (width 0.3) (layer "F.Cu") (net 5))
+  (segment (start 83.725214 91.510885) (end 82.9861 92.249999) (width 0.2) (layer "F.Cu") (net 5))
+  (segment (start 84 93.263899) (end 84 97) (width 0.3) (layer "F.Cu") (net 5))
   (segment (start 90 91.4) (end 89.889115 91.510885) (width 0.2) (layer "F.Cu") (net 5))
-  (segment (start 89.889115 91.510885) (end 83.239115 91.510885) (width 0.2) (layer "F.Cu") (net 5))
+  (segment (start 89.889115 91.510885) (end 83.725214 91.510885) (width 0.2) (layer "F.Cu") (net 5))
   (segment (start 96.30075 94.41325) (end 96.30075 92.55966) (width 0.2) (layer "F.Cu") (net 6))
   (segment (start 97.45 95.5625) (end 96.30075 94.41325) (width 0.2) (layer "F.Cu") (net 6))
