File: pcb/kitritiled.kicad_pcb (KiCad board)
At the start: 2 copper layers, 22.8 x 22.8 mm, 15 parts, among them J1 ICSP, J2 ICSP, Q1 AO3401A, Q2 AO3400A, SW1 RESET, U1 PIC12LF1571-I/SN, U2 74LVC1G123

Commit message: prefab
Other:
- board text added: "+"
- board text added: "-"
- board text added: "3V"
- board text added: "CLK"
- board text added: "DATA"
- board text added: "GND"
- board text added: "kitritiled"
- board text added: "v1"
- board text removed: "kitritiled v1"
Changed lines of the file:
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@@
     (property "Sheetfile" "kitritiled.kicad_sch")
     (property "Sheetname" "")
+    (property "exclude_from_bom" "")
     (property "ki_description" "Generic connector, single row, 01x02, script generated")
     (property "ki_keywords" "connector")
@@
     (property "Sheetfile" "kitritiled.kicad_sch")
     (property "Sheetname" "")
+    (property "exclude_from_bom" "")
     (property "ki_description" "Generic connector, single row, 01x02, script generated")
     (property "ki_keywords" "connector")
@@
       (net 5 "Net-(D1-A)") (pinfunction "A") (pintype "passive"))
     (pad "3" smd rect (at 0 0 270) (size 1.3 3.3) (layers "F.Cu" "F.Mask"))
-    (model "${KIPRJMOD}/XLamp XP-E2 XP-G2.STEP" hide
+    (model "${KIPRJMOD}/XLamp XP-E2 XP-G2.STEP"
       (offset (xyz 0 0 0.5))
-      (scale (xyz 1 1 1))
-      (rotate (xyz 0 0 90))
-    )
-    (model "${KIPRJMOD}/LED-XP-E2.stp"
-      (offset (xyz 0 0 0))
       (scale (xyz 1 1 1))
       (rotate (xyz 0 0 90))
@@
     (effects (font (size 0.8 0.8) (thickness 0.12)) (justify mirror))
   )
-  (gr_text "kitritiled\nv1" (at 90 80.5) (layer "F.SilkS")
+  (gr_text "CLK" (at 97.5 85.5 315) (layer "B.SilkS" knockout)
+    (effects (font (size 0.8 0.8) (thickness 0.1)) (justify right bottom mirror))
+  )
+  (gr_text "3V" (at 82.5 85.5 45) (layer "B.SilkS" knockout)
+    (effects (font (size 0.8 0.8) (thickness 0.1)) (justify left bottom mirror))
+  )
+  (gr_text "GND" (at 88 80 45) (layer "B.SilkS" knockout)
+    (effects (font (size 0.8 0.8) (thickness 0.1)) (justify left bottom mirror))
+  )
+  (gr_text "DATA" (at 93.5 82 315) (layer "B.SilkS" knockout)
+    (effects (font (size 0.8 0.8) (thickness 0.1)) (justify left bottom mirror))
+  )
+  (gr_text "-" (at 87 92.75) (layer "F.SilkS")
+    (effects (font (size 1 1) (thickness 0.15)) (justify left bottom))
+  )
+  (gr_text "kitritiled" (at 90 80.5) (layer "F.SilkS")
     (effects (font (size 0.8 0.8) (thickness 0.12)))
   )
+  (gr_text "v1" (at 90 100) (layer "F.SilkS")
+    (effects (font (size 0.8 0.8) (thickness 0.12)))
+  )
+  (gr_text "+" (at 87 88) (layer "F.SilkS")
+    (effects (font (size 1 1) (thickness 0.15)) (justify left bottom))
+  )
   (segment (start 94.2625 94.275) (end 93.5 94.275) (width 0.2) (layer "F.Cu") (net 1))

Commit message: jlc pn
Parts:
- C3: value 100P -> 100p
Changed lines of the file:
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@@
     (descr "SOIC, 8 Pin (JEDEC MS-012AA, https://www.analog.com/media/en/package-pcb-resources/package/pkg_pdf/soic_narrow-r/r_8.pdf), generated with kicad-footprint-generator ipc_gullwing_generator.py")
     (tags "SOIC SO")
+    (property "LCSC" "C1337248")
     (property "Sheetfile" "kitritiled.kicad_sch")
     (property "Sheetname" "")
@@
         (effects (font (size 1 1) (thickness 0.15)))
     )
-    (fp_text value "100P" (at 0 1.43 90) (layer "F.Fab")
+    (fp_text value "100p" (at 0 1.43 90) (layer "F.Fab")
         (effects (font (size 1 1) (thickness 0.15)))
     )
@@
     (tags "LED Cree XP")
     (property "DIGIKEY" "XPEBGR-L1-0000-00F02")
+    (property "LCSC" "??")
     (property "Sheetfile" "kitritiled.kicad_sch")
     (property "Sheetname" "")
@@
     (descr "SMT battery holder for CR1216/1220/1225, https://linxtechnologies.com/wp/wp-content/uploads/bat-hld-012-smt.pdf")
     (tags "battery holder coin cell cr1216 cr1220 cr1225")
-    (property "Sheetfile" "kitritiled.kicad_sch")
-    (property "Sheetname" "")
+    (property "LCSC" "C9900060949")
+    (property "Sheetfile" "kitritiled.kicad_sch")
+    (property "Sheetname" "")

Commit message: holder change
Parts:
- BT1: footprint Battery:BatteryHolder_LINX_BAT-HLD-012-SMT -> pcb:BAT_BAT-HLD-001-THM
- turned BT1 to -90 degrees
Routing:
- net +3V0: track 33.7 -> 0.00 mm, vias 2 -> 0
- net Net-(BT1-+): track 24.2 -> 0.00 mm, vias 2 -> 0
- net CLR: track 16.8 -> 0.00 mm, vias 2 -> 0
- net Net-(SW1-A): track 16.6 -> 0.00 mm
- net Net-(U1-RA4): track 14.9 -> 0.00 mm, vias 2 -> 0
- net Net-(D1-A): track 12.5 -> 0.00 mm
- net GND: track 12.1 -> 0.00 mm, vias 5 -> 0
- net Net-(Q2-G): track 7.34 -> 0.00 mm
- net Net-(U2A-RCext): track 6.53 -> 0.00 mm
- net ICSP_DATA: track 5.94 -> 0.00 mm
- net ICSP_CLK: track 3.93 -> 0.00 mm
- net Net-(Q1-G): track 3.48 -> 0.00 mm
- net Net-(U2A-Cext): track 2.04 -> 0.00 mm
Other:
- board text added: "v2"
- board text removed: "v1"

Commit message: attiny version
Parts:
- removed C1: 10u, Capacitor_SMD:C_0603_1608Metric
- removed J1, J2: ICSP, Connector_PinHeader_2.54mm:PinHeader_1x02_P2.54mm_Vertical
- added J4: AVR-ISP-6, Connector_PinHeader_1.27mm:PinHeader_2x03_P1.27mm_Vertical, F.Cu at (95.1, 83.0)
- C2: value 0.1u -> 4u7; footprint Capacitor_SMD:C_0603_1608Metric -> Capacitor_SMD:C_0402_1005Metric
- C3: footprint Capacitor_SMD:C_0603_1608Metric -> Capacitor_SMD:C_0402_1005Metric
- R2: value 59K -> 1K
- U1: value PIC12LF1571-I/SN -> ATtiny13A-SS
- moved C2 6.33 mm to (94.8, 87.3)
- moved R1 3.21 mm to (85.5, 82.5), turned to 90 degrees
- moved Q2 1.31 mm to (84.6, 95.7), turned to 90 degrees
- moved U1 1.06 mm to (98.0, 90.1)
- moved Q1 0.31 mm to (96.8, 96.3)
- turned U2 to 180 degrees
Connections:
- Q1 pad 1: Net-(Q1-G) -> /MOSI
- SW1 pad 1: Net-(SW1-A) -> /SCK
- U1 pad 1: +3V0 -> /RST
- U1 pad 2: Net-(Q1-G) -> unconnected-(U1-PB3-Pad2)
- U1 pad 3: Net-(U1-RA4) -> unconnected-(U1-PB4-Pad3)
- U1 pad 4: Net-(SW1-A) -> GND
- U1 pad 5: unconnected-(U1-RA2-Pad5) -> /MOSI
- U1 pad 6: ICSP_CLK -> /MISO
- U1 pad 7: ICSP_DATA -> /SCK
- U1 pad 8: GND -> +3V0
- U2 pad 2: Net-(U1-RA4) -> /MISO
Routing:
- net +3V0: track 0.00 -> 38.8 mm, vias 0 -> 2
- net /MISO: track 0.00 -> 25.2 mm, vias 0 -> 4
- net /SCK: track 0.00 -> 15.2 mm
- net /MOSI: track 0.00 -> 15.2 mm
- net CLR: track 0.00 -> 13.9 mm, vias 0 -> 2
- net GND: track 0.00 -> 13.8 mm, vias 0 -> 7
- net Net-(U2A-RCext): track 0.00 -> 12.8 mm, vias 0 -> 2
- net Net-(U2A-Cext): track 0.00 -> 11.1 mm
- net Net-(D1-A): track 0.00 -> 10.9 mm
- net /RST: track 0.00 -> 9.26 mm
- net Net-(BT1-+): track 0.00 -> 7.09 mm
- net Net-(Q2-G): track 0.00 -> 4.82 mm
Other:
- board text added: "JLCJLCJLCJLC"
- board text added: "kitritiled v2"
- board text removed: "3V"
- board text removed: "CLK"
- board text removed: "DATA"
- board text removed: "GND"
- board text removed: "kitritiled"
- board text removed: "v2"

Commit message: pic updates
Parts:
- removed J4: AVR-ISP-6, Connector_PinHeader_1.27mm:PinHeader_2x03_P1.27mm_Vertical
- removed U1: ATtiny13A-SS, Package_SO:SOIC-8_3.9x4.9mm_P1.27mm
- added J1: ICSP, Connector_PinHeader_1.27mm:PinHeader_1x05_P1.27mm_Vertical, F.Cu at (98.6, 85.3)
- added U3: PIC12LF1571-E/RF, Package_DFN_QFN:DFN-8-1EP_3x3mm_P0.65mm_EP1.55x2.4mm, F.Cu at (98.5, 90.0)
- moved C2 0.41 mm to (94.4, 87.4)
- moved BT1 0.10 mm to (90.1, 90.0)
Connections:
- Q1 pad 1: /MOSI -> Net-(Q1-G)
- SW1 pad 1: /SCK -> /ICSP_MCLR
- U2 pad 2: /MISO -> Net-(U2A-B)
Routing:
- net /ICSP_MCLR: track 0.00 -> 31.5 mm, vias 0 -> 4
- net Net-(BT1-+): track 7.09 -> 32.5 mm, vias 0 -> 1
- net /MISO: track 25.2 -> 0.00 mm, vias 4 -> 0
- net /SCK: track 15.2 -> 0.00 mm
- net /MOSI: track 15.2 -> 0.00 mm
- net Net-(U2A-B): track 0.00 -> 12.5 mm, vias 0 -> 2
- net /ICSP_CLK: track 0.00 -> 11.1 mm, vias 0 -> 2
- net /RST: track 9.26 -> 0.00 mm
- net /ICSP_DATA: track 0.00 -> 6.77 mm
- net Net-(Q1-G): track 0.00 -> 4.02 mm
- net +3V0: track 38.8 -> 36.5 mm, vias 2 -> 1
- net CLR: track 13.9 -> 14.9 mm
- net GND: track 13.8 -> 12.9 mm, vias 7 -> 6
Other:
- board text added: "CLK DAT GND 3V MCLR"
- board text added: "Cover after programming"
