File: pcb/kitritiled.kicad_sch (KiCad schematic)
At the start: 15 parts, among them J1 ICSP, J2 ICSP, Q1 AO3401A, Q2 AO3400A, SW1 RESET, U1 PIC12LF1571-I/SN, U2 74LVC1G123

Commit message: updates
Other:
- note added: "Misc Nets"
- note added: "Power"
- note added: "Programming"
- note added: "Tritiled"
- title: (none) -> KITRITILED
- moved on the sheet: BT1, C1, C2, C3, D1, J1, J2, L1, Q1, Q2, R1, R2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

Commit message: prefab
Parts:
- J1, J2: now left out of the parts list
Other:
- moved on the sheet: BT1, R1
Changed lines of the file:
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@@
     (fill (type none))
   )
-  (rectangle (start 16.51 17.78) (end 30.48 45.72)
+  (rectangle (start 16.51 17.145) (end 30.48 45.085)
     (stroke (width 0) (type default))
     (fill (type none))
@@
     (effects (font (size 1.27 1.27)) (justify left bottom))
   )
-  (text "Power" (at 16.51 17.78 0)
+  (text "Power" (at 16.51 17.145 0)
     (effects (font (size 1.27 1.27)) (justify left bottom))
   )
@@
     )
   )
-  (symbol (lib_id "Device:Battery_Cell") (at 20.32 35.56 0) (unit 1)
-    (in_bom yes) (on_board yes) (dnp no) (fields_autoplaced)
-    (property "Reference" "BT1" (at 24.13 32.4485 0)
-      (effects (font (size 1.27 1.27)) (justify left))
-    )
-    (property "Value" "2032" (at 24.13 34.9885 0)
-      (effects (font (size 1.27 1.27)) (justify left))
-    )
-    (property "Footprint" "Battery:BatteryHolder_LINX_BAT-HLD-012-SMT" (at 20.32 34.036 90)
-      (effects (font (size 1.27 1.27)) hide)
-    )
-    (property "Datasheet" "~" (at 20.32 34.036 90)
+  (symbol (lib_id "Device:Battery_Cell") (at 20.32 34.925 0) (unit 1)
+    (in_bom yes) (on_board yes) (dnp no) (fields_autoplaced)
+    (property "Reference" "BT1" (at 24.13 31.8135 0)
+      (effects (font (size 1.27 1.27)) (justify left))
+    )
+    (property "Value" "2032" (at 24.13 34.3535 0)
+      (effects (font (size 1.27 1.27)) (justify left))
+    )
+    (property "Footprint" "Battery:BatteryHolder_LINX_BAT-HLD-012-SMT" (at 20.32 33.401 90)
+      (effects (font (size 1.27 1.27)) hide)
+    )
+    (property "Datasheet" "~" (at 20.32 33.401 90)
       (effects (font (size 1.27 1.27)) hide)
     )
@@
   )
   (symbol (lib_id "Connector:Conn_01x02_Pin") (at 24.13 71.12 0) (unit 1)
-    (in_bom yes) (on_board yes) (dnp no)
+    (in_bom no) (on_board yes) (dnp no)
     (property "Reference" "J2" (at 21.59 71.12 0)
       (effects (font (size 1.27 1.27)))
@@
   )
   (symbol (lib_id "Connector:Conn_01x02_Pin") (at 24.13 62.23 0) (mirror x) (unit 1)
-    (in_bom yes) (on_board yes) (dnp no) (fields_autoplaced)
+    (in_bom no) (on_board yes) (dnp no) (fields_autoplaced)
     (property "Reference" "J1" (at 22.86 59.69 0)
       (effects (font (size 1.27 1.27)) (justify right))
@@
     )
   )
-  (symbol (lib_id "power:GND") (at 20.32 38.1 0) (unit 1)
-    (in_bom yes) (on_board yes) (dnp no) (fields_autoplaced)
-    (property "Reference" "#PWR06" (at 20.32 44.45 0)
-      (effects (font (size 1.27 1.27)) hide)
-    )
-    (property "Value" "GND" (at 20.32 43.18 0)
-      (effects (font (size 1.27 1.27)))
-    )
-    (property "Footprint" "" (at 20.32 38.1 0)
-      (effects (font (size 1.27 1.27)) hide)
-    )
-    (property "Datasheet" "" (at 20.32 38.1 0)
+  (symbol (lib_id "power:GND") (at 20.32 37.465 0) (unit 1)
+    (in_bom yes) (on_board yes) (dnp no) (fields_autoplaced)
+    (property "Reference" "#PWR06" (at 20.32 43.815 0)
+      (effects (font (size 1.27 1.27)) hide)
+    )
+    (property "Value" "GND" (at 20.32 42.545 0)
+      (effects (font (size 1.27 1.27)))
+    )
+    (property "Footprint" "" (at 20.32 37.465 0)
+      (effects (font (size 1.27 1.27)) hide)
+    )
+    (property "Datasheet" "" (at 20.32 37.465 0)
       (effects (font (size 1.27 1.27)) hide)
     )
@@
     )
   )
-  (symbol (lib_id "power:+3V0") (at 20.32 25.4 0) (unit 1)
-    (in_bom yes) (on_board yes) (dnp no) (fields_autoplaced)
-    (property "Reference" "#PWR01" (at 20.32 29.21 0)
-      (effects (font (size 1.27 1.27)) hide)
-    )
-    (property "Value" "+3V0" (at 20.32 20.32 0)
-      (effects (font (size 1.27 1.27)))
-    )
-    (property "Footprint" "" (at 20.32 25.4 0)
-      (effects (font (size 1.27 1.27)) hide)
-    )
-    (property "Datasheet" "" (at 20.32 25.4 0)
+  (symbol (lib_id "power:+3V0") (at 20.32 24.765 0) (unit 1)
+    (in_bom yes) (on_board yes) (dnp no) (fields_autoplaced)
+    (property "Reference" "#PWR01" (at 20.32 28.575 0)
+      (effects (font (size 1.27 1.27)) hide)
+    )
+    (property "Value" "+3V0" (at 20.32 19.685 0)
+      (effects (font (size 1.27 1.27)))
+    )
+    (property "Footprint" "" (at 20.32 24.765 0)
+      (effects (font (size 1.27 1.27)) hide)
+    )
+    (property "Datasheet" "" (at 20.32 24.765 0)
       (effects (font (size 1.27 1.27)) hide)
     )
@@
     )
   )
-  (symbol (lib_id "Device:R_Small") (at 20.32 27.94 0) (unit 1)
-    (in_bom yes) (on_board yes) (dnp no) (fields_autoplaced)
-    (property "Reference" "R1" (at 22.86 26.67 0)
-      (effects (font (size 1.27 1.27)) (justify left))
-    )
-    (property "Value" "100" (at 22.86 29.21 0)
-      (effects (font (size 1.27 1.27)) (justify left))
-    )
-    (property "Footprint" "Resistor_SMD:R_0402_1005Metric" (at 20.32 27.94 0)
-      (effects (font (size 1.27 1.27)) hide)
-    )
-    (property "Datasheet" "~" (at 20.32 27.94 0)
-      (effects (font (size 1.27 1.27)) hide)
-    )
-    (property "LCSC" "C25076" (at 20.32 27.94 0)
-      (effects (font (size 1.27 1.27)) hide)
-    )
+  (symbol (lib_id "Device:R_Small") (at 20.32 27.305 0) (unit 1)
+    (in_bom yes) (on_board yes) (dnp no) (fields_autoplaced)
+    (property "Reference" "R1" (at 22.86 26.035 0)
+      (effects (font (size 1.27 1.27)) (justify left))
+    )
+    (property "Value" "100" (at 22.86 28.575 0)
+      (effects (font (size 1.27 1.27)) (justify left))
+    )
+    (property "Footprint" "Resistor_SMD:R_0402_1005Metric" (at 20.32 27.305 0)
+      (effects (font (size 1.27 1.27)) hide)
+    )
+    (property "Datasheet" "~" (at 20.32 27.305 0)
+      (effects (font (size 1.27 1.27)) hide)
+    )
+    (property "LCSC" "C25076" (at 20.32 27.305 0)
+      (effects (font (size 1.27 1.27)) hide)
+    )

Commit message: jlc pn
Parts:
- BT1: LCSC (none) -> C9900060949
- C3: value 100P -> 100p
- D1: LCSC (none) -> ??
- U1: LCSC (none) -> C1337248
Changed lines of the file:
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@@
+      (effects (font (size 1.27 1.27)) hide)
+    )
+    (property "LCSC" "C9900060949" (at 20.32 34.925 0)
       (effects (font (size 1.27 1.27)) hide)
     )
@@
       (effects (font (size 1.27 1.27)) hide)
     )
+    (property "LCSC" "??" (at 183.515 52.705 90)
+      (effects (font (size 1.27 1.27)) hide)
+    )
     (pin "1")
     (pin "2")
@@
   (symbol (lib_id "Device:C_Small") (at 135.255 65.405 90) (unit 1)
     (in_bom yes) (on_board yes) (dnp no) (fields_autoplaced)
-    (property "Reference" "C3" (at 135.2613 59.055 90)
-      (effects (font (size 1.27 1.27)))
-    )
-    (property "Value" "100P" (at 135.2613 61.595 90)
+    (property "Reference" "C3" (at 135.2613 58.42 90)
+      (effects (font (size 1.27 1.27)))
+    )
+    (property "Value" "100p" (at 135.2613 60.96 90)
       (effects (font (size 1.27 1.27)))
     )
@@
       (effects (font (size 1.27 1.27)) hide)
     )
+    (property "LCSC" "C1337248" (at 89.535 60.325 0)
+      (effects (font (size 1.27 1.27)) hide)
+    )

Commit message: fix part number
Parts:
- BT1: LCSC C9900060949 -> (none)
- D1: LCSC ?? -> C9900060949
Changed lines of the file:
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@@
       (effects (font (size 1.27 1.27)) hide)
     )
-    (property "LCSC" "C9900060949" (at 20.32 34.925 0)
+    (property "LCSC" "" (at 20.32 34.925 0)
       (effects (font (size 1.27 1.27)) hide)
     )
@@
       (effects (font (size 1.27 1.27)) hide)
     )
-    (property "LCSC" "??" (at 183.515 52.705 90)
+    (property "LCSC" "C9900060949" (at 183.515 52.705 90)
       (effects (font (size 1.27 1.27)) hide)
     )

Commit message: holder change
Parts:
- BT1: footprint Battery:BatteryHolder_LINX_BAT-HLD-012-SMT -> pcb:BAT_BAT-HLD-001-THM
Changed lines of the file:
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@@
       (effects (font (size 1.27 1.27)) (justify left))
     )
-    (property "Footprint" "Battery:BatteryHolder_LINX_BAT-HLD-012-SMT" (at 20.32 33.401 90)
+    (property "Footprint" "pcb:BAT_BAT-HLD-001-THM" (at 20.32 33.401 90)
       (effects (font (size 1.27 1.27)) hide)
     )

Commit message: attiny version
Parts:
- removed C1: 10u, Capacitor_SMD:C_0603_1608Metric, symbol Device:C_Small
- removed J1, J2: ICSP, Connector_PinHeader_2.54mm:PinHeader_1x02_P2.54mm_Vertical, symbol Connector:Conn_01x02_Pin
- removed U1: PIC12LF1571-I/SN, Package_SO:SOIC-8_3.9x4.9mm_P1.27mm, symbol MCU_Microchip_PIC12:PIC12LF1501-IMS
- added J4: AVR-ISP-6, Connector_PinHeader_1.27mm:PinHeader_2x03_P1.27mm_Vertical, symbol Connector:AVR-ISP-6
- added U1: ATtiny13A-SS, Package_SO:SOIC-8_3.9x4.9mm_P1.27mm, symbol MCU_Microchip_ATtiny:ATtiny13A-SS
- C2: value 0.1u -> 4u7; footprint Capacitor_SMD:C_0603_1608Metric -> Capacitor_SMD:C_0402_1005Metric; LCSC C14663 -> C23733
- C3: footprint Capacitor_SMD:C_0603_1608Metric -> Capacitor_SMD:C_0402_1005Metric; LCSC C14858 -> C1546
- R2: value 59K -> 1K; LCSC C321568 -> C11702
Connections:
- net +3V0: now also J4.2 (VCC), U1.8 (VCC)
- net GND: now also J4.6 (GND), U1.4 (GND)
- net MOSI: now reaches Q1.1 (G)
- net MOSI: now also J4.4 (MOSI), U1.5 (PB0)
- net MISO: now reaches U2.2 (B)
- net MISO: now also J4.1 (MISO), U1.6 (PB1)
- net SCK: now reaches SW1.1 (A)
- net SCK: now also J4.3 (SCK), U1.7 (PB2)
- new net RST: J4.5 (~{RST}), U1.1 (~{RESET}/PB5)
- no-connect marks 1 -> 2
Other:
- moved on the sheet: BT1, C2, C3, D1, L1, Q1, Q2, R1, R2, SW1, U2A, U2B

Commit message: pic updates
Parts:
- removed J4: AVR-ISP-6, Connector_PinHeader_1.27mm:PinHeader_2x03_P1.27mm_Vertical, symbol Connector:AVR-ISP-6
- removed U1: ATtiny13A-SS, Package_SO:SOIC-8_3.9x4.9mm_P1.27mm, symbol MCU_Microchip_ATtiny:ATtiny13A-SS
- added J1: ICSP, Connector_PinHeader_1.27mm:PinHeader_1x05_P1.27mm_Vertical, symbol Connector:Conn_PIC_ICSP_ICD
- added U3: PIC12LF1571-E/RF, Package_DFN_QFN:DFN-8-1EP_3x3mm_P0.65mm_EP1.55x2.4mm, symbol MCU_Microchip_PIC12:PIC12LF1501-xMC
Connections:
- net +3V0: now also J1.2 (VDD), U3.1 (VDD)
- net GND: now also J1.3 (VSS), U3.8 (VSS)
- net MISO: no longer names the net of U2.2 (B)
- net MISO: now also U3.3 (RA4)
- net MOSI: no longer names the net of Q1.1 (G)
- net MOSI: now also U3.2 (RA5)
- net SCK renamed ICSP_MCLR
- net ICSP_MCLR: now also J1.1 (~{MCLR}/VPP), U3.4 (RA3)
- new net ICSP_CLK: J1.5 (PGC/ICSPCLK), U3.6 (RA1)
- new net ICSP_DATA: J1.4 (PGD/ICSPDAT), U3.7 (RA0)
Other:
- moved on the sheet: BT1, C2, C3, D1, L1, Q1, Q2, R1, R2, SW1, U2A, U2B
